Commit message: it works now I think

File: zau2_description/urdf/astra.urdf.xacro (robot description, xacro)
@@ -1,5 +1,5 @@
 <?xml version="1.0"?>
 <robot name="sensor_astra" xmlns:xacro="http://ros.org/wiki/xacro">
-  <xacro:include filename="$(find zau2_description)/urdf/ur.gazebo.xacro" />
+  <xacro:include filename="$(find ur_e_description)/urdf/ur.gazebo.xacro" />
   <!-- Xacro properties -->
   <xacro:property name="astra_cam_py" value="-0.0125" />
@@ -56,5 +56,5 @@
         <origin xyz="0.0 0.0 -0.03" rpy="${pi/2} 0 0" />
         <geometry>
-          <mesh filename="package://zau2_description/meshes/sensors/astra2.dae" scale="1 1 1" />
+          <mesh filename="package://t2rgb_description/meshes/sensors/astra2.dae" scale="1 1 1" />
         </geometry>
       </visual>

File: zau2_description/urdf/moving_base_odom.urdf.xacro (robot description, xacro)
@@ -1,9 +1,10 @@
 <?xml version="1.0"?>
-<robot name="moving_base" xmlns:xacro="http://ros.org/wiki/xacro">
-    <xacro:include filename="$(find zau2_description)/urdf/properties.xacro" />
-    <xacro:include filename="$(find zau2_description)/urdf/moving_base_odom.gazebo.xacro" />
+<robot xmlns:xacro="http://ros.org/wiki/xacro" name="zau2">
+    <!-- properties file -->
+    <xacro:include filename="$(find zau2_description)/urdf/properties.xacro"/>
     <xacro:property name="M_PI" value="3.1415926535897931" />
-    <!-- testing adding a velodyne laser  -->
-    <!-- VLP-16 -->
+    <!-- gazebo.xacro files -->
+    <xacro:include filename="$(find zau2_description)/urdf/moving_base_odom.gazebo.xacro"/>
+    <!-- ######################## sensors ######################## -->
     <!-- velodyne -->
     <xacro:arg name="gpu" default="false" />
@@ -16,6 +17,5 @@
         <origin xyz="-0.350 0.050 0.850" rpy="0 0 0" />
     </xacro:VLP-16>
-    <!-- velodyne -->
-    <!-- testing adding a sensor camera -->
+    <!-- RGB camera -->
     <xacro:include filename="$(find zau2_description)/urdf/astra.urdf.xacro" />
     <xacro:sensor_astra parent="base_link_mb" prefix="camera_mb">
@@ -23,6 +23,5 @@
             rpy="0 0 3.14" />
     </xacro:sensor_astra>
-    <!-- testing adding a sensor camera -->
-    <!-- add intel realsense camera d415 sensor -->
+    <!-- intel realsense camera d415 sensor -->
     <xacro:arg name="realsense_enabled" default="$(optenv REALSENSE_ENABLED 1)" />
     <xacro:arg name="realsense_topic" default="$(optenv REALSENSE_TOPIC realsense)" />
@@ -45,5 +44,4 @@
             parent_link="$(arg realsense_prefix)_realsense_mountpoint" />
     </xacro:if>
-    <!-- add intel realsense d415 sensor -->
     <!-- add intel realsense l515 camera -->
     <xacro:arg name="use_nominal_extrinsics" default="false" />
@@ -55,5 +53,4 @@
         <origin xyz="0.350 0.180 0.850" rpy="0 0 0" />
     </xacro:sensor_l515>
-    <!-- add intel realsense l515 camera -->
     <!-- add intel realsense t265 -->
     <xacro:include filename="$(find realsense_ros_gazebo)/xacro/tracker.xacro" />
@@ -61,6 +58,8 @@
         <origin rpy="0 0 0" xyz="0.350 0.060 0.860" />
     </xacro:realsense_T265>
-    <!-- add intel realsense t265 -->
+    <!-- ######################## the actual robot ######################## -->
+    <!-- world link -->
     <link name="base_footprint" />
+    <!-- the mobile base link and joint to the world -->
     <joint name="base_joint" type="fixed">
         <parent link="base_footprint" />
@@ -72,8 +71,5 @@
             <origin xyz="-0.43 -0.33 0.03" rpy="1.57 0 1.57" />
             <geometry>
-                <!-- <box size="0.900 0.600 0.770" /> -->
-                <!-- <box size="0.900 0.650 0.770" /> -->
-                <mesh filename="package://zau2_description/meshes/moving_base/moving_base.STL"
-                    scale="0.001 0.001 0.001" />
+                <mesh filename="package://zau2_description/meshes/moving_base/moving_base.STL" scale="0.001 0.001 0.001" />
             </geometry>
             <material name="light_black" />
@@ -91,6 +87,5 @@
             <mass value="500" />
             <origin xyz="-0.00065 -0.085 0.062" />
-            <inertia ixx="0.6022" ixy="-0.02364" ixz="-0.1197" iyy="1.7386" iyz="-0.001544"
-                izz="2.0296" />
+            <inertia ixx="0.6022" ixy="-0.02364" ixz="-0.1197" iyy="1.7386" iyz="-0.001544" izz="2.0296" />
         </inertial>
     </link>
@@ -100,5 +95,5 @@
         <child link="inertial_link" />
     </joint>
-    <!-- #################### wheels #################### -->
+    <!-- wheels -->
     <joint name="wheel_left_joint" type="continuous">
         <parent link="base_link_mb" />
@@ -138,5 +133,5 @@
             <origin xyz="0 0 0.055" rpy="1.57 0 0" />
             <geometry>
-                <mesh filename="package://zau2_description/meshes/wheels/left_tire.stl"
+                <mesh filename="package://ur_e_description/meshes/wheels/left_tire.stl"
                     scale="0.0025 0.0025 0.0025" />
             </geometry>
@@ -167,5 +162,4 @@
                 <mesh filename="package://zau2_description/meshes/wheels/left_tire.stl"
                     scale="0.0020 0.0020 0.0020" />
-                <!-- <cylinder length="0.024" radius="0.084" /> -->
             </geometry>
             <material name="dark" />
@@ -196,5 +190,4 @@
                 <mesh filename="package://zau2_description/meshes/wheels/left_tire.stl"
                     scale="0.0020 0.0020 0.0020" />
-                <!-- <cylinder length="0.024" radius="0.084" /> -->
             </geometry>
             <material name="dark" />
@@ -214,5 +207,4 @@
         </inertial>
     </link>
-    <!-- back caster -->
     <!-- front caster -->
     <joint name="caster_front_right_joint" type="fixed">
@@ -227,5 +219,4 @@
                 <mesh filename="package://zau2_description/meshes/wheels/left_tire.stl"
                     scale="0.0020 0.0020 0.0020" />
-                <!-- <cylinder length="0.024" radius="0.084" /> -->
             </geometry>
             <material name="dark" />
@@ -256,5 +247,4 @@
                 <mesh filename="package://zau2_description/meshes/wheels/left_tire.stl"
                     scale="0.0020 0.0020 0.0020" />
-                <!-- <cylinder length="0.024" radius="0.084" /> -->
             </geometry>
             <material name="dark" />
@@ -274,5 +264,5 @@
         </inertial>
     </link>
-    <!-- front caster -->
+    <!-- imu -->
     <joint name="imu_joint" type="fixed">
         <parent link="base_link_mb" />
@@ -300,5 +290,4 @@
         </inertial>
     </link>
-    <!-- lidar sensor front -->
     <!-- lidar sensor back -->
     <joint name="scan_joint_back" type="fixed">
@@ -320,4 +309,3 @@
         </inertial>
     </link>
-    <!-- lidar sensor back -->
 </robot>

File: zau2_description/urdf/realsense/_l515.urdf.xacro (robot description, xacro)
@@ -8,5 +8,5 @@
 <robot name="sensor_l515" xmlns:xacro="http://ros.org/wiki/xacro">
   <!-- Includes -->
-  <xacro:include filename="$(find zau2_description)/urdf/realsense/_l515.gazebo.xacro" />
+  <xacro:include filename="$(find ur_e_description)/urdf/realsense/_l515.gazebo.xacro" />
   <xacro:include filename="$(find realsense2_description)/urdf/_materials.urdf.xacro" />
   <xacro:include filename="$(find realsense2_description)/urdf/_usb_plug.urdf.xacro" /> <!-- this

File: zau2_description/urdf/zau2.urdf.xacro (robot description, xacro)
@@ -1,11 +1,9 @@
 <?xml version="1.0"?>
-<robot xmlns:xacro="http://ros.org/wiki/xacro"
-  name="ur5e">
-  <!-- common stuff -->
-  <xacro:include filename="$(find zau2_description)/urdf/common.gazebo.xacro" />
-  <!-- ur5e -->
-  <xacro:include filename="$(find zau2_description)/urdf/ur5e.urdf.xacro" />
-  <!-- arm -->
-  <xacro:ur5e_robot prefix="" joint_limited="true"
+<robot xmlns:xacro="http://ros.org/wiki/xacro" name="zau2">
+    <xacro:include filename="$(find zau2_description)/urdf/common.gazebo.xacro" />
+    <!-- ur5e -->
+    <xacro:include filename="$(find zau2_description)/urdf/my_ur5e_macro.urdf.xacro" />
+    <!-- arm -->
+    <xacro:ur5e_robot prefix="" joint_limited="true"
     shoulder_pan_lower_limit="${-pi}" shoulder_pan_upper_limit="${pi}"
     shoulder_lift_lower_limit="${-pi}" shoulder_lift_upper_limit="${pi}"
@@ -14,4 +12,4 @@
     wrist_2_lower_limit="${-pi}" wrist_2_upper_limit="${pi}"
     wrist_3_lower_limit="${-pi}" wrist_3_upper_limit="${pi}"
-  />
+    />
 </robot>

Commit message: fixed some deps

File: zau2_description/urdf/astra.urdf.xacro (robot description, xacro)
@@ -1,5 +1,5 @@
 <?xml version="1.0"?>
 <robot name="sensor_astra" xmlns:xacro="http://ros.org/wiki/xacro">
-  <xacro:include filename="$(find ur_e_description)/urdf/ur.gazebo.xacro" />
+  <xacro:include filename="$(find zau2_description)/urdf/ur.gazebo.xacro" />
   <!-- Xacro properties -->
   <xacro:property name="astra_cam_py" value="-0.0125" />
@@ -56,5 +56,5 @@
         <origin xyz="0.0 0.0 -0.03" rpy="${pi/2} 0 0" />
         <geometry>
-          <mesh filename="package://t2rgb_description/meshes/sensors/astra2.dae" scale="1 1 1" />
+          <mesh filename="package://zau2_description/meshes/sensors/astra2.dae" scale="1 1 1" />
         </geometry>
       </visual>
