Commit message: trying on mmtzau

File: zau2_description/urdf/properties.xacro (robot description, xacro)
@@ -1,17 +1,12 @@
-<?xml version="1.0" ?>
+<?xml version="1.0"?>
 <robot name="properties" xmlns:xacro="http://ros.org/wiki/xacro">
-    <!--Read common properties from turtlebot3 and then add missing stuff-->
-    <!--    <xacro:include filename="$(find turtlebot3_description)/urdf/common_properties.xacro"/>-->
-    <material name="Yellow">
-        <color rgba="1.0 1.0 0.0 1.0"/>
+    <material name="grey">
+        <color rgba="0.7 0.7 0.7 1.0" />
     </material>
-    <material name="Orange">
-        <color rgba="1.0 0.4 0.0 1.0"/>
+    <material name="dark">
+        <color rgba="0.3 0.3 0.3 1.0" />
     </material>
-    <material name="grey">
-        <color rgba="0.7 0.7 0.7 1.0"/>
-    </material>
-    <material name="Pink">
-        <color rgba="1 0 0.8 1.0"/>
+    <material name="light_black">
+        <color rgba="0.4 0.4 0.4 1.0" />
     </material>
 </robot>
