Commit message: running into some issues

File: zau2_description/urdf/moving_base_odom.urdf.xacro (robot description, xacro)
@@ -34,5 +34,5 @@
         <color rgba="1.0 1.0 1.0 1.0" />
     </material>
-    <xacro:include filename="$(find ur_e_description)/urdf/realsense/intel_realsense.urdf.xacro" />
+    <xacro:include filename="$(find zau2_description)/urdf/realsense/intel_realsense.urdf.xacro" />
     <xacro:if value="$(arg realsense_enabled)">
         <link name="$(arg realsense_prefix)_realsense_mountpoint" />
@@ -50,5 +50,5 @@
     <xacro:arg name="add_plug" default="false" />
     <xacro:arg name="use_mesh" default="true" />
-    <xacro:include filename="$(find ur_e_description)/urdf/realsense/_l515.urdf.xacro" />
+    <xacro:include filename="$(find zau2_description)/urdf/realsense/_l515.urdf.xacro" />
     <xacro:sensor_l515 parent="base_link_mb" use_nominal_extrinsics="$(arg use_nominal_extrinsics)"
         add_plug="$(arg add_plug)" use_mesh="$(arg use_mesh)">
@@ -74,5 +74,5 @@
                 <!-- <box size="0.900 0.600 0.770" /> -->
                 <!-- <box size="0.900 0.650 0.770" /> -->
-                <mesh filename="package://ur_e_description/meshes/moving_base/moving_base.STL"
+                <mesh filename="package://zau2_description/meshes/moving_base/moving_base.STL"
                     scale="0.001 0.001 0.001" />
             </geometry>
@@ -111,5 +111,5 @@
             <origin xyz="0 0 -0.055" rpy="-1.57 0 0" />
             <geometry>
-                <mesh filename="package://ur_e_description/meshes/wheels/left_tire.stl"
+                <mesh filename="package://zau2_description/meshes/wheels/left_tire.stl"
                     scale="0.0025 0.0025 0.0025" />
             </geometry>
@@ -138,5 +138,5 @@
             <origin xyz="0 0 0.055" rpy="1.57 0 0" />
             <geometry>
-                <mesh filename="package://ur_e_description/meshes/wheels/left_tire.stl"
+                <mesh filename="package://zau2_description/meshes/wheels/left_tire.stl"
                     scale="0.0025 0.0025 0.0025" />
             </geometry>
@@ -165,5 +165,5 @@
             <origin xyz="0.027 -0.06 0" rpy="1.57 0 0" />
             <geometry>
-                <mesh filename="package://ur_e_description/meshes/wheels/left_tire.stl"
+                <mesh filename="package://zau2_description/meshes/wheels/left_tire.stl"
                     scale="0.0020 0.0020 0.0020" />
                 <!-- <cylinder length="0.024" radius="0.084" /> -->
@@ -194,5 +194,5 @@
             <origin xyz="0.027 -0.06 0" rpy="-1.57 0 0" />
             <geometry>
-                <mesh filename="package://ur_e_description/meshes/wheels/left_tire.stl"
+                <mesh filename="package://zau2_description/meshes/wheels/left_tire.stl"
                     scale="0.0020 0.0020 0.0020" />
                 <!-- <cylinder length="0.024" radius="0.084" /> -->
@@ -225,5 +225,5 @@
             <origin xyz="0 -0.06 0" rpy="1.57 0 0" />
             <geometry>
-                <mesh filename="package://ur_e_description/meshes/wheels/left_tire.stl"
+                <mesh filename="package://zau2_description/meshes/wheels/left_tire.stl"
                     scale="0.0020 0.0020 0.0020" />
                 <!-- <cylinder length="0.024" radius="0.084" /> -->
@@ -254,5 +254,5 @@
             <origin xyz="0 -0.06 0" rpy="-1.57 0 0" />
             <geometry>
-                <mesh filename="package://ur_e_description/meshes/wheels/left_tire.stl"
+                <mesh filename="package://zau2_description/meshes/wheels/left_tire.stl"
                     scale="0.0020 0.0020 0.0020" />
                 <!-- <cylinder length="0.024" radius="0.084" /> -->

File: zau2_description/urdf/ur5e.urdf.xacro (robot description, xacro)
@@ -106,13 +106,13 @@
       <visual>
         <geometry>
-          <mesh filename="package://ur_e_description/meshes/ur5e/visual/base.dae" />
-        </geometry>
-        <material name="LightGrey">
-          <color rgba="0.7 0.7 0.7 1.0" />
-        </material>
-      </visual>
-      <collision>
-        <geometry>
-          <mesh filename="package://ur_e_description/meshes/ur5e/collision/base.stl" />
+          <mesh filename="package://zau2_description/meshes/ur5e/visual/base.dae" />
+        </geometry>
+        <material name="LightGrey">
+          <color rgba="0.7 0.7 0.7 1.0" />
+        </material>
+      </visual>
+      <collision>
+        <geometry>
+          <mesh filename="package://zau2_description/meshes/ur5e/collision/base.stl" />
         </geometry>
       </collision>
@@ -148,13 +148,13 @@
       <visual>
         <geometry>
-          <mesh filename="package://ur_e_description/meshes/ur5e/visual/shoulder.dae" />
-        </geometry>
-        <material name="LightGrey">
-          <color rgba="0.7 0.7 0.7 1.0" />
-        </material>
-      </visual>
-      <collision>
-        <geometry>
-          <mesh filename="package://ur_e_description/meshes/ur5e/collision/shoulder.stl" />
+          <mesh filename="package://zau2_description/meshes/ur5e/visual/shoulder.dae" />
+        </geometry>
+        <material name="LightGrey">
+          <color rgba="0.7 0.7 0.7 1.0" />
+        </material>
+      </visual>
+      <collision>
+        <geometry>
+          <mesh filename="package://zau2_description/meshes/ur5e/collision/shoulder.stl" />
         </geometry>
       </collision>
@@ -190,13 +190,13 @@
       <visual>
         <geometry>
-          <mesh filename="package://ur_e_description/meshes/ur5e/visual/upperarm.dae" />
-        </geometry>
-        <material name="LightGrey">
-          <color rgba="0.7 0.7 0.7 1.0" />
-        </material>
-      </visual>
-      <collision>
-        <geometry>
-          <mesh filename="package://ur_e_description/meshes/ur5e/collision/upperarm.stl" />
+          <mesh filename="package://zau2_description/meshes/ur5e/visual/upperarm.dae" />
+        </geometry>
+        <material name="LightGrey">
+          <color rgba="0.7 0.7 0.7 1.0" />
+        </material>
+      </visual>
+      <collision>
+        <geometry>
+          <mesh filename="package://zau2_description/meshes/ur5e/collision/upperarm.stl" />
         </geometry>
       </collision>
@@ -232,13 +232,13 @@
       <visual>
         <geometry>
-          <mesh filename="package://ur_e_description/meshes/ur5e/visual/forearm.dae" />
-        </geometry>
-        <material name="LightGrey">
-          <color rgba="0.7 0.7 0.7 1.0" />
-        </material>
-      </visual>
-      <collision>
-        <geometry>
-          <mesh filename="package://ur_e_description/meshes/ur5e/collision/forearm.stl" />
+          <mesh filename="package://zau2_description/meshes/ur5e/visual/forearm.dae" />
+        </geometry>
+        <material name="LightGrey">
+          <color rgba="0.7 0.7 0.7 1.0" />
+        </material>
+      </visual>
+      <collision>
+        <geometry>
+          <mesh filename="package://zau2_description/meshes/ur5e/collision/forearm.stl" />
         </geometry>
       </collision>
@@ -274,13 +274,13 @@
       <visual>
         <geometry>
-          <mesh filename="package://ur_e_description/meshes/ur5e/visual/wrist1.dae" />
-        </geometry>
-        <material name="LightGrey">
-          <color rgba="0.7 0.7 0.7 1.0" />
-        </material>
-      </visual>
-      <collision>
-        <geometry>
-          <mesh filename="package://ur_e_description/meshes/ur5e/collision/wrist1.stl" />
+          <mesh filename="package://zau2_description/meshes/ur5e/visual/wrist1.dae" />
+        </geometry>
+        <material name="LightGrey">
+          <color rgba="0.7 0.7 0.7 1.0" />
+        </material>
+      </visual>
+      <collision>
+        <geometry>
+          <mesh filename="package://zau2_description/meshes/ur5e/collision/wrist1.stl" />
         </geometry>
       </collision>
@@ -316,13 +316,13 @@
       <visual>
         <geometry>
-          <mesh filename="package://ur_e_description/meshes/ur5e/visual/wrist2.dae" />
-        </geometry>
-        <material name="LightGrey">
-          <color rgba="0.7 0.7 0.7 1.0" />
-        </material>
-      </visual>
-      <collision>
-        <geometry>
-          <mesh filename="package://ur_e_description/meshes/ur5e/collision/wrist2.stl" />
+          <mesh filename="package://zau2_description/meshes/ur5e/visual/wrist2.dae" />
+        </geometry>
+        <material name="LightGrey">
+          <color rgba="0.7 0.7 0.7 1.0" />
+        </material>
+      </visual>
+      <collision>
+        <geometry>
+          <mesh filename="package://zau2_description/meshes/ur5e/collision/wrist2.stl" />
         </geometry>
       </collision>
@@ -358,13 +358,13 @@
       <visual>
         <geometry>
-          <mesh filename="package://ur_e_description/meshes/ur5e/visual/wrist3.dae" />
-        </geometry>
-        <material name="LightGrey">
-          <color rgba="0.7 0.7 0.7 1.0" />
-        </material>
-      </visual>
-      <collision>
-        <geometry>
-          <mesh filename="package://ur_e_description/meshes/ur5e/collision/wrist3.stl" />
+          <mesh filename="package://zau2_description/meshes/ur5e/visual/wrist3.dae" />
+        </geometry>
+        <material name="LightGrey">
+          <color rgba="0.7 0.7 0.7 1.0" />
+        </material>
+      </visual>
+      <collision>
+        <geometry>
+          <mesh filename="package://zau2_description/meshes/ur5e/collision/wrist3.stl" />
         </geometry>
       </collision>
@@ -396,5 +396,5 @@
       <visual>
         <geometry>
-          <mesh filename="package://ur_e_description/meshes/ur5e/visual/weiss-mount.dae" />
+          <mesh filename="package://zau2_description/meshes/ur5e/visual/weiss-mount.dae" />
         </geometry>
         <origin xyz="-0.071 0 0" rpy="${pi/-2.0} 0 ${pi/-2.0}" />
@@ -402,5 +402,5 @@
       <visual>
         <geometry>
-          <mesh filename="package://ur_e_description/meshes/ur5e/visual/weiss-cg.dae" />
+          <mesh filename="package://zau2_description/meshes/ur5e/visual/weiss-cg.dae" />
         </geometry>
         <origin xyz="-0.07 0 0" rpy="${pi/-2.0} 0 ${pi/-2.0}" />
@@ -487,5 +487,5 @@
     ur.gazebo.xacro
     ur5e.urdf.xacro -->
-    <xacro:include filename="$(find ur_e_description)/urdf/astra.urdf.xacro" />
+    <xacro:include filename="$(find zau2_description)/urdf/astra.urdf.xacro" />
     <xacro:sensor_astra parent="ee_link" prefix="camera">
       <origin xyz="0.06 -0.05 0.05"

Commit message: fixing some deps

File: zau2_description/urdf/moving_base_odom.urdf.xacro (robot description, xacro)
@@ -133,5 +133,5 @@
             <origin xyz="0 0 0.055" rpy="1.57 0 0" />
             <geometry>
-                <mesh filename="package://ur_e_description/meshes/wheels/left_tire.stl"
+                <mesh filename="package://zau2_description/meshes/wheels/left_tire.stl"
                     scale="0.0025 0.0025 0.0025" />
             </geometry>

Commit message: it's done. finally done.

File: zau2_description/urdf/moving_base_odom.urdf.xacro (robot description, xacro)
@@ -60,8 +60,8 @@
     <!-- ######################## the actual robot ######################## -->
     <!-- world link -->
-    <link name="base_footprint" />
+    <!-- <link name="base_footprint" /> -->
     <!-- the mobile base link and joint to the world -->
     <joint name="base_joint" type="fixed">
-        <parent link="base_footprint" />
+        <parent link="world" /> <!-- Changed parent link to world for zau2 -->
         <child link="base_link_mb" />
         <origin xyz="0 0 0.010" rpy="0 0 0" />

File: zau2_description/urdf/properties.xacro (robot description, xacro)
@@ -1,7 +1,7 @@
 <?xml version="1.0"?>
 <robot name="properties" xmlns:xacro="http://ros.org/wiki/xacro">
-    <material name="grey">
+    <!-- <material name="grey">
         <color rgba="0.7 0.7 0.7 1.0" />
-    </material>
+    </material> -->
     <material name="dark">
         <color rgba="0.3 0.3 0.3 1.0" />

File: zau2_description/urdf/zau2.urdf.xacro (robot description, xacro)
@@ -42,6 +42,6 @@
     <!-- <xacro:table_macro name="table" parent="world" width="${table_width}"
                        lenght="${table_lenght}" height="${table_height}"
-                       tabletop_thickness="${table_tabletop_thickness}" leg_radius="${table_leg_radius}"> -->
-        <!-- <origin xyz="-1 0 0" rpy="0 0 ${M_PI/2}" /> -->
+                       tabletop_thickness="${table_tabletop_thickness}" leg_radius="${table_leg_radius}">
+        <origin xyz="-1 0 0" rpy="0 0 ${M_PI/2}" /> -->
     <!-- </xacro:table_macro> -->
     <!-- Place AGV -->
@@ -60,8 +60,8 @@
     />
     <!--  Place robot on top of the table1-->
-    <joint name="tabletop_table_to_ur10e" type="fixed">
+    <joint name="moving_base_to_ur10e" type="fixed">
         <parent link="base_link_mb" />
         <child link = "base_link"/>
-        <origin xyz="0.0 0.0 0.001" rpy="0.0 0.0 0.0" />
+        <origin xyz="-0.296 -0.1688 0.826" rpy="0.0 0.0 0.0" />
     </joint>
     <!-- Place hand camera 1 in the scene-->
@@ -79,5 +79,5 @@
     <!-- Put world camera on top of tripod -->
     <!-- <xacro:sensor_astra prefix="world_camera" parent="tripod_right_support"> -->
-        <!-- <origin xyz="0.02 0.07 0.015" rpy="0 0.0 0" /> -->
+        <!-- <origin xyz="0.02 0.07 0.015   " rpy="0 0.0 0" /> -->
     <!-- </xacro:sensor_astra> -->
 </robot>

Commit message: fixed tf tree, teleop now works

File: zau2_description/urdf/moving_base_odom.urdf.xacro (robot description, xacro)
@@ -60,8 +60,8 @@
     <!-- ######################## the actual robot ######################## -->
     <!-- world link -->
-    <!-- <link name="base_footprint" /> -->
+    <link name="base_footprint" />
     <!-- the mobile base link and joint to the world -->
     <joint name="base_joint" type="fixed">
-        <parent link="world" /> <!-- Changed parent link to world for zau2 -->
+        <parent link="base_footprint" /> <!-- Changed parent link to world for zau2 -->
         <child link="base_link_mb" />
         <origin xyz="0 0 0.010" rpy="0 0 0" />

File: zau2_description/urdf/zau2.urdf.xacro (robot description, xacro)
@@ -38,5 +38,5 @@
     <!-- Declare links and joints -->
     <!-- ####################################### -->
-    <link name="world"/>
+    <!-- <link name="base_footprint"/> -->
     <!-- Place table 1 in the scene-->
     <!-- <xacro:table_macro name="table" parent="world" width="${table_width}"
