Commit message: calib done https://github.com/lardemua/atom/issues/627

File: zau2_calibration/urdf/optimized/optimized_2023_11_09-08_23_12_PM.urdf.xacro (robot description, xacro)
@@ -326,5 +326,5 @@
   </gazebo>
   <joint name="camera_mb_rgb_joint" type="fixed">
-    <origin xyz="-0.0005939912475418017 -0.020760752691411064 0.004606006358523848" rpy="-7.154213722272843e-05 0.0014393055442115453 -0.001256399799057782"/>
+    <origin xyz="-0.00268690097733682 -0.02211102392368211 0.00933903152732468" rpy="0.0013667588694060034 0.003374884660056257 -0.004380415573102704"/>
     <parent link="camera_mb_link"/>
     <child link="camera_mb_rgb_frame"/>
@@ -1341,5 +1341,5 @@
   </gazebo>
   <joint name="moving_base_to_ur10e" type="fixed">
-    <origin xyz="-0.2996402976116742 -0.173470205216959 0.8164851176351837" rpy="0.019212793338771322 -0.006824817943325027 0.004172540492778811"/>
+    <origin xyz="-0.29080828236738887 -0.17318700651125601 0.8141083786235186" rpy="0.009544800566189504 -0.006807856359061044 0.00191945984086278"/>
     <parent link="base_link_mb"/>
     <child link="base_link"/>
@@ -1367,5 +1367,5 @@
   </gazebo>
   <joint name="hand_camera_rgb_joint" type="fixed">
-    <origin xyz="-0.010154441666284 -0.04045840412698659 0.0021193421556219274" rpy="0.019726555450851814 -0.006704900716282688 0.0029485996806694554"/>
+    <origin xyz="-0.00587961940719331 -0.04032641828730139 0.011640372363261113" rpy="0.011695562337120607 -0.006308160685743149 0.0016664506737826496"/>
     <parent link="hand_camera_link"/>
     <child link="hand_camera_rgb_frame"/>

File: zau2_calibration/urdf/optimized/optimized_2023_11_09-08_23_27_PM.urdf.xacro (robot description, xacro)
@@ -326,5 +326,5 @@
   </gazebo>
   <joint name="camera_mb_rgb_joint" type="fixed">
-    <origin xyz="-0.0005939912475418017 -0.020760752691411064 0.004606006358523848" rpy="-7.154213722272843e-05 0.0014393055442115453 -0.001256399799057782"/>
+    <origin xyz="-0.001934987366326906 -0.022418393111488612 0.009216240678672445" rpy="0.0012256793791603374 0.0032537123608355452 -0.0031318897888562448"/>
     <parent link="camera_mb_link"/>
     <child link="camera_mb_rgb_frame"/>
@@ -1341,5 +1341,5 @@
   </gazebo>
   <joint name="moving_base_to_ur10e" type="fixed">
-    <origin xyz="-0.2996402976116742 -0.173470205216959 0.8164851176351837" rpy="0.019212793338771322 -0.006824817943325027 0.004172540492778811"/>
+    <origin xyz="-0.29251385618213266 -0.1733078870574534 0.8154957255122318" rpy="0.009003945468375664 -0.007840350943944809 0.002381386363494842"/>
     <parent link="base_link_mb"/>
     <child link="base_link"/>
@@ -1367,5 +1367,5 @@
   </gazebo>
   <joint name="hand_camera_rgb_joint" type="fixed">
-    <origin xyz="-0.010154441666284 -0.04045840412698659 0.0021193421556219274" rpy="0.019726555450851814 -0.006704900716282688 0.0029485996806694554"/>
+    <origin xyz="-0.007298526550409437 -0.040197399689916376 0.009448634641550244" rpy="0.010853583898898176 -0.007270073820663751 0.00194697885292813"/>
     <parent link="hand_camera_link"/>
     <child link="hand_camera_rgb_frame"/>

File: zau2_calibration/urdf/optimized/optimized_2023_11_09-08_24_37_PM.urdf.xacro (robot description, xacro)
@@ -326,5 +326,5 @@
   </gazebo>
   <joint name="camera_mb_rgb_joint" type="fixed">
-    <origin xyz="-0.0005939912475418017 -0.020760752691411064 0.004606006358523848" rpy="-7.154213722272843e-05 0.0014393055442115453 -0.001256399799057782"/>
+    <origin xyz="-0.0005900676893641255 -0.02011542903994364 0.00444420892701465" rpy="-0.0001069415233400011 0.0014514670102202998 -0.001243245869713526"/>
     <parent link="camera_mb_link"/>
     <child link="camera_mb_rgb_frame"/>
@@ -1341,5 +1341,5 @@
   </gazebo>
   <joint name="moving_base_to_ur10e" type="fixed">
-    <origin xyz="-0.2996402976116742 -0.173470205216959 0.8164851176351837" rpy="0.019212793338771322 -0.006824817943325027 0.004172540492778811"/>
+    <origin xyz="-0.29963017823166116 -0.17363378543944888 0.8164209689506127" rpy="0.019426854824260334 -0.006665912145439311 0.004233148779700565"/>
     <parent link="base_link_mb"/>
     <child link="base_link"/>
@@ -1367,5 +1367,5 @@
   </gazebo>
   <joint name="hand_camera_rgb_joint" type="fixed">
-    <origin xyz="-0.010154441666284 -0.04045840412698659 0.0021193421556219274" rpy="0.019726555450851814 -0.006704900716282688 0.0029485996806694554"/>
+    <origin xyz="-0.0099818829042447 -0.04008003000929472 0.002065211380138149" rpy="0.019897775583555093 -0.006568860849537548 0.0029730326951418577"/>
     <parent link="hand_camera_link"/>
     <child link="hand_camera_rgb_frame"/>
