Commit message: updated some things

File: zau2_calibration/urdf/optimized/optimized_2023_11_13-02_31_46_PM.urdf.xacro (robot description, xacro)
@@ -326,5 +326,5 @@
   </gazebo>
   <joint name="camera_mb_rgb_joint" type="fixed">
-    <origin xyz="0.001181661512279207 -0.02233414753759305 0.017900054866000468" rpy="-9.519310431952304e-05 0.0017527078719506205 -0.00011166613355385859"/>
+    <origin xyz="0.0029982341478304625 -0.15453141044581947 0.0017631992519028584" rpy="-0.15300400259892513 -0.05103956061701438 0.04043798245474575"/>
     <parent link="camera_mb_link"/>
     <child link="camera_mb_rgb_frame"/>
@@ -1341,5 +1341,5 @@
   </gazebo>
   <joint name="moving_base_to_ur10e" type="fixed">
-    <origin xyz="-0.2987863929766694 -0.17761590227475765 0.8420208540664372" rpy="0.0002276608168357014 0.0028645564569913648 0.002980079967480762"/>
+    <origin xyz="-0.06550430969077946 -0.20068140562708303 0.7701607522847277" rpy="0.008495222528992761 -0.06476246636879816 0.08681673672203193"/>
     <parent link="base_link_mb"/>
     <child link="base_link"/>
@@ -1367,5 +1367,5 @@
   </gazebo>
   <joint name="hand_camera_rgb_joint" type="fixed">
-    <origin xyz="0.0005300496919829319 -0.03305326841714277 -0.0011765094246307852" rpy="0.0006653166628127665 0.003190483626357427 -0.0018251628023147246"/>
+    <origin xyz="0.11080552095497179 -0.09180984023596526 0.019518793203476985" rpy="-0.10956723318375611 -0.11221015975369078 -0.10579912807267902"/>
     <parent link="hand_camera_link"/>
     <child link="hand_camera_rgb_frame"/>

File: zau2_calibration/urdf/optimized/optimized_2023_11_13-02_44_16_PM.urdf.xacro (robot description, xacro)
@@ -326,5 +326,5 @@
   </gazebo>
   <joint name="camera_mb_rgb_joint" type="fixed">
-    <origin xyz="0.001181661512279207 -0.02233414753759305 0.017900054866000468" rpy="-9.519310431952304e-05 0.0017527078719506205 -0.00011166613355385859"/>
+    <origin xyz="7.944477159212925e-05 -0.02403523855761391 -0.006164324933969467" rpy="0.00031739097039905904 0.0016537277340836771 -0.0023575426989979205"/>
     <parent link="camera_mb_link"/>
     <child link="camera_mb_rgb_frame"/>
@@ -1341,5 +1341,5 @@
   </gazebo>
   <joint name="moving_base_to_ur10e" type="fixed">
-    <origin xyz="-0.2987863929766694 -0.17761590227475765 0.8420208540664372" rpy="0.0002276608168357014 0.0028645564569913648 0.002980079967480762"/>
+    <origin xyz="-0.21977891525014573 -0.17597599762218255 0.7843514188484013" rpy="-0.00021044628608432844 0.0032659067908771136 0.0035454172220537226"/>
     <parent link="base_link_mb"/>
     <child link="base_link"/>
@@ -1367,5 +1367,5 @@
   </gazebo>
   <joint name="hand_camera_rgb_joint" type="fixed">
-    <origin xyz="0.0005300496919829319 -0.03305326841714277 -0.0011765094246307852" rpy="0.0006653166628127665 0.003190483626357427 -0.0018251628023147246"/>
+    <origin xyz="0.061256378341678436 -0.035742286474154186 0.06178401467375801" rpy="0.002430854006463132 0.003940967724314861 -0.005415237285532533"/>
     <parent link="hand_camera_link"/>
     <child link="hand_camera_rgb_frame"/>

File: zau2_calibration/urdf/optimized/optimized_2023_11_13-02_44_29_PM.urdf.xacro (robot description, xacro)
@@ -326,5 +326,5 @@
   </gazebo>
   <joint name="camera_mb_rgb_joint" type="fixed">
-    <origin xyz="0.001181661512279207 -0.02233414753759305 0.017900054866000468" rpy="-9.519310431952304e-05 0.0017527078719506205 -0.00011166613355385859"/>
+    <origin xyz="0.00017198590608283074 -0.02399804701441123 0.003531569674462413" rpy="0.0002973318202129127 0.0017504902277658723 -0.0024913012558411985"/>
     <parent link="camera_mb_link"/>
     <child link="camera_mb_rgb_frame"/>
@@ -1341,5 +1341,5 @@
   </gazebo>
   <joint name="moving_base_to_ur10e" type="fixed">
-    <origin xyz="-0.2987863929766694 -0.17761590227475765 0.8420208540664372" rpy="0.0002276608168357014 0.0028645564569913648 0.002980079967480762"/>
+    <origin xyz="-0.2962720078781006 -0.18005647760400528 0.8189653924561735" rpy="-0.0011126828721519987 0.0030286517952701282 0.0037136223847478965"/>
     <parent link="base_link_mb"/>
     <child link="base_link"/>
@@ -1367,5 +1367,5 @@
   </gazebo>
   <joint name="hand_camera_rgb_joint" type="fixed">
-    <origin xyz="0.0005300496919829319 -0.03305326841714277 -0.0011765094246307852" rpy="0.0006653166628127665 0.003190483626357427 -0.0018251628023147246"/>
+    <origin xyz="8.104828366454178e-05 -0.03378995358334403 0.00930632692023276" rpy="0.0017292349246432837 0.0037351566459406143 -0.006200655796837794"/>
     <parent link="hand_camera_link"/>
     <child link="hand_camera_rgb_frame"/>

File: zau2_calibration/urdf/optimized/optimized_2023_11_13-03_14_59_PM.urdf.xacro (robot description, xacro)
@@ -326,5 +326,5 @@
   </gazebo>
   <joint name="camera_mb_rgb_joint" type="fixed">
-    <origin xyz="0.001181661512279207 -0.02233414753759305 0.017900054866000468" rpy="-9.519310431952304e-05 0.0017527078719506205 -0.00011166613355385859"/>
+    <origin xyz="-8.850155593433403e-05 -0.02371418540230728 0.04452771745200986" rpy="0.001438707371573749 -0.0012306866876347414 -0.0032986756302610886"/>
     <parent link="camera_mb_link"/>
     <child link="camera_mb_rgb_frame"/>
@@ -1341,5 +1341,5 @@
   </gazebo>
   <joint name="moving_base_to_ur10e" type="fixed">
-    <origin xyz="-0.2987863929766694 -0.17761590227475765 0.8420208540664372" rpy="0.0002276608168357014 0.0028645564569913648 0.002980079967480762"/>
+    <origin xyz="-0.2366062658190607 -0.20454322580468226 0.8566224356186781" rpy="0.0257492993945461 0.003475107739342993 -0.007744853996551299"/>
     <parent link="base_link_mb"/>
     <child link="base_link"/>
@@ -1367,5 +1367,5 @@
   </gazebo>
   <joint name="hand_camera_rgb_joint" type="fixed">
-    <origin xyz="0.0005300496919829319 -0.03305326841714277 -0.0011765094246307852" rpy="0.0006653166628127665 0.003190483626357427 -0.0018251628023147246"/>
+    <origin xyz="0.05502183128404345 -0.08691124787983125 0.026751410029680484" rpy="0.023801878860340055 -0.0005781208679610546 0.014495033017129545"/>
     <parent link="hand_camera_link"/>
     <child link="hand_camera_rgb_frame"/>

File: zau2_calibration/urdf/optimized/optimized_2023_11_15-06_32_52_PM.urdf.xacro (robot description, xacro)
@@ -326,5 +326,5 @@
   </gazebo>
   <joint name="camera_mb_rgb_joint" type="fixed">
-    <origin xyz="0.001181661512279207 -0.02233414753759305 0.017900054866000468" rpy="-9.519310431952304e-05 0.0017527078719506205 -0.00011166613355385859"/>
+    <origin xyz="-0.0001934854571290495 -0.023260518421514043 0.00707938135926764" rpy="0.0001891672406931857 0.0021986463200907554 -0.0016441898262149583"/>
     <parent link="camera_mb_link"/>
     <child link="camera_mb_rgb_frame"/>
@@ -1341,5 +1341,5 @@
   </gazebo>
   <joint name="moving_base_to_ur10e" type="fixed">
-    <origin xyz="-0.2987863929766694 -0.17761590227475765 0.8420208540664372" rpy="0.0002276608168357014 0.0028645564569913648 0.002980079967480762"/>
+    <origin xyz="-0.2983325063928416 -0.17422379330284582 0.8290823650217436" rpy="-0.0003033054388993645 0.0030343448062713912 -0.00048352116752864037"/>
     <parent link="base_link_mb"/>
     <child link="base_link"/>
@@ -1367,5 +1367,5 @@
   </gazebo>
   <joint name="hand_camera_rgb_joint" type="fixed">
-    <origin xyz="0.0005300496919829319 -0.03305326841714277 -0.0011765094246307852" rpy="0.0006653166628127665 0.003190483626357427 -0.0018251628023147246"/>
+    <origin xyz="-0.0004157860285595804 -0.0319254624199588 0.0006997966144269256" rpy="-0.00043390293498459545 0.0033209903408423303 0.0005654851799050853"/>
     <parent link="hand_camera_link"/>
     <child link="hand_camera_rgb_frame"/>
