Commit message: some missing adjustments to the new description package

File: zau2_real_calib/urdf/initial_estimate.urdf.xacro (robot description, xacro)
@@ -46,5 +46,5 @@
     <!-- </xacro:table_macro> -->
     <!-- Place AGV -->
-    <xacro:include filename="$(find zau2_description)/urdf/moving_base_odom.urdf.xacro" />
+    <xacro:include filename="$(find zau2_real_description)/urdf/moving_base_odom.urdf.xacro" />
     <!--  Place manipulator1 in the scene-->
     <xacro:ur_robot_gazebo

File: zau2_real_description/urdf/astra.urdf.xacro (robot description, xacro)
@@ -1,5 +1,5 @@
 <?xml version="1.0"?>
 <robot name="sensor_astra" xmlns:xacro="http://ros.org/wiki/xacro">
-  <xacro:include filename="$(find zau2_description)/urdf/ur.gazebo.xacro" />
+  <xacro:include filename="$(find zau2_real_description)/urdf/ur.gazebo.xacro" />
   <!-- Xacro properties -->
   <xacro:property name="astra_cam_py" value="-0.0125" />
@@ -56,5 +56,5 @@
         <origin xyz="0.0 0.0 -0.03" rpy="${pi/2} 0 0" />
         <geometry>
-          <mesh filename="package://zau2_description/meshes/sensors/astra2.dae" scale="1 1 1" />
+          <mesh filename="package://zau2_real_description/meshes/sensors/astra2.dae" scale="1 1 1" />
         </geometry>
       </visual>

File: zau2_real_description/urdf/realsense/_l515.urdf.xacro (robot description, xacro)
@@ -8,5 +8,5 @@
 <robot name="sensor_l515" xmlns:xacro="http://ros.org/wiki/xacro">
   <!-- Includes -->
-  <xacro:include filename="$(find zau2_description)/urdf/realsense/_l515.gazebo.xacro" />
+  <xacro:include filename="$(find zau2_real_description)/urdf/realsense/_l515.gazebo.xacro" />
   <xacro:include filename="$(find realsense2_description)/urdf/_materials.urdf.xacro" />
   <xacro:include filename="$(find realsense2_description)/urdf/_usb_plug.urdf.xacro" /> <!-- this
