Commit message: eliminated some extra sensors in the real description

File: zau2_real_description/urdf/moving_base_odom.urdf.xacro (robot description, xacro)
@@ -8,5 +8,5 @@
     <!-- ######################## sensors ######################## -->
     <!-- velodyne -->
-    <xacro:arg name="gpu" default="false" />
+    <!-- <xacro:arg name="gpu" default="false" />
     <xacro:property name="gpu" value="$(arg gpu)" />
     <xacro:arg name="organize_cloud" default="false" />
@@ -16,5 +16,5 @@
         organize_cloud="${organize_cloud}" hz="10" samples="440" gpu="${gpu}">
         <origin xyz="-0.350 0.050 0.850" rpy="0 0 0" />
-    </xacro:VLP-16>
+    </xacro:VLP-16> -->
     <!-- RGB camera -->
     <xacro:include filename="$(find zau2_real_description)/urdf/astra.urdf.xacro" />
@@ -24,14 +24,14 @@
     </xacro:sensor_astra>
     <!-- intel realsense camera d415 sensor -->
-    <xacro:arg name="realsense_enabled" default="$(optenv REALSENSE_ENABLED 1)" />
+    <!-- <xacro:arg name="realsense_enabled" default="$(optenv REALSENSE_ENABLED 1)" />
     <xacro:arg name="realsense_topic" default="$(optenv REALSENSE_TOPIC realsense)" />
     <xacro:arg name="realsense_prefix" default="$(optenv REALSENSE_PREFIX camera_realsense)" />
     <xacro:arg name="realsense_parent" default="$(optenv REALSENSE_PARENT base_link_mb)" />
     <xacro:arg name="realsense_xyz" default="$(optenv REALSENSE_XYZ 0.350 -0.180 0.850)" />
-    <xacro:arg name="realsense_rpy" default="$(optenv REALSENSE_RPY 0 0 0)" />
-    <material name="white">
+    <xacro:arg name="realsense_rpy" default="$(optenv REALSENSE_RPY 0 0 0)" /> -->
+    <!-- <material name="white">
         <color rgba="1.0 1.0 1.0 1.0" />
-    </material>
-    <xacro:include filename="$(find zau2_real_description)/urdf/realsense/intel_realsense.urdf.xacro" />
+    </material> -->
+    <!-- <xacro:include filename="$(find zau2_real_description)/urdf/realsense/intel_realsense.urdf.xacro" />
     <xacro:if value="$(arg realsense_enabled)">
         <link name="$(arg realsense_prefix)_realsense_mountpoint" />
@@ -43,7 +43,7 @@
         <xacro:intel_realsense_mount prefix="$(arg realsense_prefix)" topic="$(arg realsense_topic)"
             parent_link="$(arg realsense_prefix)_realsense_mountpoint" />
-    </xacro:if>
+    </xacro:if> -->
     <!-- add intel realsense l515 camera -->
-    <xacro:arg name="use_nominal_extrinsics" default="false" />
+    <!-- <xacro:arg name="use_nominal_extrinsics" default="false" />
     <xacro:arg name="add_plug" default="false" />
     <xacro:arg name="use_mesh" default="true" />
@@ -52,10 +52,10 @@
         add_plug="$(arg add_plug)" use_mesh="$(arg use_mesh)">
         <origin xyz="0.350 0.180 0.850" rpy="0 0 0" />
-    </xacro:sensor_l515>
+    </xacro:sensor_l515> -->
     <!-- add intel realsense t265 -->
-    <xacro:include filename="$(find realsense_ros_gazebo)/xacro/tracker.xacro" />
+    <!-- <xacro:include filename="$(find realsense_ros_gazebo)/xacro/tracker.xacro" />
     <xacro:realsense_T265 sensor_name="camera_t265" parent_link="base_link_mb" rate="30.0">
         <origin rpy="0 0 0" xyz="0.350 0.060 0.860" />
-    </xacro:realsense_T265>
+    </xacro:realsense_T265> -->
     <!-- ######################## the actual robot ######################## -->
     <!-- world link -->
